File: NinjaScanPseudo.brd (EAGLE design)
At the start: 25.4 x 35.6 mm, 57 parts, among them CON2 ZX62-B-5PA(11), CON3 JST_SH-12SM, IC1 LTC3550EDHC, IC2 MPU-6000, IC4 MAG3110FCR, J1 JUMPER1608, U1 DM3AT-SF-PEJM5, U2 H.FL, U3 NEO-6T, U4 MS5611-01BA01

Commit message: some wiring issues were fixed.
Parts:
- removed C14, C15, C17, C18, C19, C20, C22, C24: 0.1u, additional:1005
- removed C16: 1u, additional:1005
- removed C21, C23: 2.2u, additional:1005
- removed CON1: (no value), additional:JST_ZH-2B(MM)
- removed CON2: ZX62-B-5PA(11), additional:ZX62-AB-5PA
- removed CON3: JST_SH-12SM, additional:JST_SH-SM12B
- removed IC1: LTC3550EDHC, main:DFN16BP
- removed IC2: MPU-6000, sensor:QFN24
- removed IC4: MAG3110FCR, main:DFN10
- removed J1: JUMPER1608, additional:1608
- removed L1: 2.2u, additional:3225
- removed L2: LQG15HS27NJ02, additional:1005
- removed LED3: LED3, mami_pero:1608
- removed LED4: 1608(LED), mami_pero:1608
- removed R10, R11: 10K, additional:1005
- removed R8: 10, additional:1005
- removed R9: pull-down, additional:1005
- removed U1: DM3AT-SF-PEJM5, additional:DM3
- removed U2: H.FL, gps:H.FL
- removed U3: NEO-6T, gps:NEO
- removed U4: MS5611-01BA01, sensor:LGA8
- added R13, R14: 10k, mami_pero:1005
- added U$1: LTC3550, mami_pero:DFN-16
- added U$10: NEO-6, mami_pero:NEO-6
- added U$11: LQG15HS, mami_pero:LQG15HS
- added U$12: HIROSE_H.FL, mami_pero:HIROSE_H.FL
- added U$13: JST_SH_12, mami_pero:JST_SH_12
- added U$14: OMRON_B3U_1000P, mami_pero:B3U_1000P
- added U$16: 2200p, mami_pero:1005
- added U$17, U$18, U$19, U$23, U$24, U$25, U$27, U$28: 0.1u, mami_pero:1005
- added U$2: 2.2u, mami_pero:LQH32CN
- added U$20: pull-down, mami_pero:1005
- added U$21: 10, mami_pero:1005
- added U$22: 0, mami_pero:1005
- added U$26: 1u, mami_pero:1005
- added U$29: 3216(CAP), mami_pero:3216
- added U$3: JST_ZR_2, mami_pero:JST_ZR_2
- added U$30: 4.7u, mami_pero:2012
- added U$31: 330k, mami_pero:1608
- added U$32, U$33: 1608(LED), mami_pero:1608
- added U$36: FA128, mami_pero:FA128
- added U$4: MICRO_USB, mami_pero:MICRO_USB
- added U$5: DM3A, mami_pero:DM3A
- added U$7: MS5611-01BA03, mami_pero:MS5611
- added U$9: STM32F405_64, mami_pero:TQFP-64
- C1: value 10u -> 0.1u; device additional:3216 -> mami_pero:1005
- C10, C11: value 0.1u -> 8p; device additional:1005 -> mami_pero:1005
- C12, C13: value 0.1u -> 0,1u; device additional:1005 -> mami_pero:1005
- C2, C3, C5, C6: device additional:1005 -> mami_pero:1005
- C4: value 4.7u -> 0.1u; device additional:2012 -> mami_pero:1005
- C7: value 2200p -> 0,1u; device additional:1005 -> mami_pero:1005
- C8, C9: value 0.1u -> 2.2u; device additional:1005 -> mami_pero:1005
- LED1, LED2: value (none) -> 1608(LED); device additional:1608D -> mami_pero:1608
- R1, R2: value 1K -> 1k; device additional:1005 -> mami_pero:1005
- R3, R4: value 2K -> 2k; device additional:1005 -> mami_pero:1005
- R5: value 1.24K -> 1.24k; device additional:1005 -> mami_pero:1005
- R6: value 604K -> 604k; device additional:1005 -> mami_pero:1005
- R7: value 150K -> 150k; device additional:1005 -> mami_pero:1005
- U$15: value 330k -> 0.1u
- U$6: value STM32F405_64 -> MPU6000; device mami_pero:TQFP-64 -> mami_pero:QFN24
- U$8: value OMRON_B3U_1000P -> MAG3110; device mami_pero:B3U_1000P -> mami_pero:MAG3110
- moved C9 85.0 mm to (-49.5, 49.5), flipped to the top
- moved C13 84.9 mm to (-53.3, -17.8), flipped to the top, turned to 0 degrees
- moved C11 77.2 mm to (-53.3, -10.2), turned to 0 degrees
- moved C10 77.1 mm to (-53.3, -6.35), flipped to the top
- moved C7 76.4 mm to (-41.9, 49.5), flipped to the top, turned to 0 degrees
- moved C12 76.2 mm to (-53.3, -14.0)
- moved C4 62.9 mm to (-30.5, 49.5), flipped to the top
- moved C8 61.5 mm to (-45.7, 49.5), flipped to the top, turned to 0 degrees
- moved C6 61.2 mm to (-38.1, 49.5)
- moved U$35 59.4 mm to (-47.0, 45.7), turned to 0 degrees
- moved U$6 59.2 mm to (-33.0, 35.6), turned to 0 degrees
- moved U$34 57.3 mm to (-43.2, 45.7), turned to 0 degrees
- moved U$15 56.9 mm to (-29.2, 40.6), turned to 0 degrees
- moved U$8 55.6 mm to (-25.4, 40.6), turned to 0 degrees
- moved C1 54.3 mm to (-19.1, 49.5), flipped to the top, turned to 0 degrees
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Connections:
- removed net +3V: C1.2, C11.P$1, C12.P$1, C15.P$2, C16.P$2, C17.P$2, C18.P$1, C19.P$1, C20.P$2, C22.P$1, C24.P$1, C5.P$2, C6.P$2, C8.P$2, C9.P$1, CON3.3, IC2.13, IC4.2, IC4.8, L1.2, R10.P$1, R11.P$1, R6.P$1, U$15.P$2, U$6.P$1, U$6.P$13, U$6.P$19, U$6.P$32, U$6.P$48, U$6.P$64, U1.4, U3.23, U4.1, U4.2
- removed net -INT0: U3.3
- removed net GPS_USB_VBUS: R9.P$2, U3.7
- removed net IMU_-CS: IC2.8
- removed net IMU_SCK: IC2.23, U$6.P$51
- removed net SMB0_SCL: IC2.7, IC4.7, R11.P$2, U4.8
- removed net SMB0_SDA: IC2.6, IC4.6, R10.P$2, U4.7
- removed net SPI1_CS: U$6.P$20, U1.2
- removed net SPI1_MISO: U$6.P$22, U1.7
- removed net SPI1_MOSI: U$6.P$23, U1.3
- removed net SPI1_SCLK: U$6.P$21, U1.5
- removed net USB_VBUS: C2.P$2, CON2.1, IC1.1
- new net +3V3: C1.P$2, C12.P$2, C13.P$2, C4.P$2, C5.P$2, C6.P$2, C7.P$2, R13.P$2, R14.P$2, R6.P$2, U$10.23, U$15.P$2, U$18.P$2, U$19.P$2, U$2.P$2, U$25.P$2, U$26.P$2, U$27.P$2, U$28.P$2, U$29.P$2, U$31.P$2, U$5.4, U$6.13, U$7.P$1, U$7.P$2, U$8.P$2, U$8.P$8, U$9.P$1, U$9.P$13, U$9.P$19, U$9.P$32, U$9.P$48, U$9.P$64
- new net +5V: C2.P$2, U$1.1, U$4.1
- new net -INT: U$10.3
- new net AUX_MAG_SCL: R14.P$1, U$6.7, U$7.P$8, U$8.P$7
- new net AUX_MAG_SDA: R13.P$1, U$6.6, U$7.P$7, U$8.P$6
- new net GPS_USB_VBAS: U$10.7, U$20.P$2
- new net IMU_INTR: U$6.12
- new net IMU_SCLK: U$6.23, U$9.P$21
- new net N$23: C10.P$2, U$36.1, U$9.P$5
- new net N$24: C11.P$2, U$36.3, U$9.P$6
- new net SPI3_CS: U$5.2, U$9.P$50
- new net SPI3_MISO: U$5.7, U$9.P$52
- new net SPI3_MOSI: U$5.3, U$9.P$53
- new net SPI3_SCK: U$5.5, U$9.P$51
- net AGND: now also U$10.10, U$10.12, U$10.24, U$12.GND@1, U$12.GND@2, U$12.GND@3, U$22.P$1; no longer J1.P$1, U2.GND@1, U2.GND@2, U2.GND@3, U3.10, U3.12, U3.13
- net GND: now also C1.P$1, C10.P$1, C11.P$1, C12.P$1, C3.P$1, C4.P$1, C7.P$1, C9.P$1, R3.P$1, R4.P$1, R5.P$1, R7.P$1, U$1.8, U$1.9, U$1.P$17, U$10.13, U$14.P$1, U$15.P$1, U$16.P$1, U$18.P$1, U$19.P$1, U$20.P$1, U$22.P$2, U$23.P$1, U$24.P$1, U$25.P$1, U$26.P$1, U$27.P$1, U$28.P$1, U$29.P$1, U$3.P$1, U$30.1, U$4.5, U$5.6, U$5.GND@1, U$5.GND@2, U$5.GND@3, U$5.GND@4, U$6.1, U$6.11, U$6.18, U$7.P$3, U$7.P$4, U$8.P$10, U$8.P$5, U$9.P$12, U$9.P$18, U$9.P$63; no longer C1.1, C10.P$2, C11.P$2, C12.P$2, C14.P$1, C15.P$1, C16.P$1, C17.P$1, C18.P$2, C19.P$2, C20.P$1, C21.P$1, C22.P$2, C23.P$1, C24.P$2, C3.P$2, C4.1, C7.P$2, C9.P$2, CON1.2, CON2.5, CON2.GUIDE@L1, CON2.GUIDE@L3, CON2.GUIDE@R1, CON2.GUIDE@R3, CON3.2, CON3.4, CON3.GUIDE@L, CON3.GUIDE@R, IC1.17, IC1.8, IC1.9, IC2.1, IC2.11, IC2.18, IC4.10, IC4.5, J1.P$2, R3.P$2, R4.P$2, R5.P$2, R7.P$2, R9.P$1, U$6.P$12, U$6.P$18, U$6.P$63, U$8.P$1, U1.6, U1.GND@1, U1.GND@2, U1.GND@3, U1.GND@4, U3.24, U4.3, U4.4
- net GPIO1: now also U$9.P$24; no longer U$6.P$24
- net GPIO2: now also U$9.P$25; no longer U$6.P$25
- net GPS_BKUP: now also U$10.22; no longer U3.22
- net GPS_RX: now also U$10.20, U$9.P$38; no longer U$6.P$38, U3.20
- net GPS_TX: now also U$10.21, U$9.P$37; no longer U$6.P$37, U3.21
- net GPS_USB_D+: now also U$10.6; no longer U3.6
- net GPS_USB_D-: now also U$10.5; no longer U3.5
- net I2C1_SCL: now also U$9.P$61; no longer CON3.6, U$6.P$61
- net I2C1_SDA: now also U$9.P$62; no longer CON3.5, U$6.P$62
- net I2C2_SCL: now also U$9.P$29; no longer U$6.P$29
- net I2C2_SDA: now also U$9.P$30; no longer U$6.P$30
- net IMU_CS: now also U$6.8, U$9.P$20; no longer U$6.P$50
- net IMU_MISO: now also U$6.9, U$9.P$22; no longer IC2.9, U$6.P$52
- net IMU_MOSI: now also U$6.24, U$9.P$23; no longer IC2.24, U$6.P$53
- net N$1: now also U$1.10, U$2.P$1; no longer C10.P$1, IC2.10
- net N$10: now also LED2.P$2, R2.P$2; no longer LED4.P$2, U$35.P$2
- net N$11: now also U$33.P$1, U$9.P$35; no longer LED2.K, R2.P$1
- net N$12: now also U$32.P$2, U$34.P$2; no longer IC1.2, R3.P$1
- net N$13: now also U$16.P$2, U$6.20; no longer IC1.3, R4.P$1
- net N$14: now also U$17.P$2, U$6.10; no longer IC1.14, R5.P$1
- net N$15: now also U$10.11, U$11.P$2, U$12.SIG; no longer C5.P$1, IC1.6, R6.P$2, R7.P$1
- net N$16: now also U$24.P$2, U$8.P$4; no longer IC1.5, R1.P$2
- net N$17: now also U$23.P$2, U$8.P$1; no longer IC1.10, L1.1
- net N$18: now also U$10.8, U$10.9, U$21.P$2; no longer IC1.4, R2.P$2
- net N$19: now also U$11.P$1, U$21.P$1; no longer C4.2, CON1.1, IC1.11, IC1.15, IC1.7, LED1.A, LED2.A
- net N$2: now also R3.P$2, U$1.2; no longer C23.P$2, U$6.P$31
- net N$20: now also U$32.P$1, U$9.P$36; no longer LED3.P$1, U$6.P$36
- net N$21: now also U$14.P$2, U$31.P$1, U$9.P$7; no longer U$15.P$1, U$6.P$7, U$8.P$2
- net N$22: now also U$33.P$2, U$35.P$2; no longer C13.P$2, IC4.1
- net N$29: now also C8.P$2, U$9.P$31; no longer C14.P$2, IC4.4
- net N$3: now also R4.P$2, U$1.3; no longer C7.P$1, IC2.20
- net N$31: now also C9.P$2, U$9.P$47; no longer C21.P$2, U$6.P$47
- net N$4: now also R5.P$2, U$1.14; no longer LED4.P$1, U$6.P$35
- net N$5: now also LED1.P$1, LED2.P$1, U$1.11, U$1.15, U$1.7, U$3.P$2, U$30.2; no longer LED3.P$2, U$34.P$2
- net N$6: now also C5.P$1, R7.P$2, U$1.6; no longer L2.P$1, R8.P$1
- net N$7: now also R1.P$1, U$1.5; no longer L2.P$2, U2.SIG, U3.11
- net N$8: now also LED1.P$2, R1.P$2; no longer R8.P$2, U3.8, U3.9
- net N$9: now also R2.P$1, U$1.4; no longer LED1.K, R1.P$1
- net SWDCLK: now also U$9.P$49; no longer CON3.11, U$6.P$49
- net SWDIO: now also U$9.P$46; no longer CON3.12, U$6.P$46
- net USART1_RX: now also U$9.P$59; no longer CON3.8, U$6.P$59
- net USART1_TX: now also U$9.P$58; no longer CON3.7, U$6.P$58
- net USB_D+: now also U$4.3, U$9.P$45; no longer CON2.3, U$6.P$45
- net USB_D-: now also U$4.2, U$9.P$44; no longer CON2.2, U$6.P$44
- net USB_ID: now also U$4.4; no longer CON2.4
- net VCC: now also C3.P$2, U$1.16; no longer C3.P$1, CON3.1, IC1.16
Routing:
- net +3V: track 169.0 -> 0.00 mm, vias 13 -> 0
- net VCC: track 54.9 -> 0.00 mm, vias 3 -> 0
- net I2C1_SDA: track 40.6 -> 0.00 mm
- net I2C1_SCL: track 39.5 -> 0.00 mm
- net USART1_RX: track 34.0 -> 0.00 mm, vias 2 -> 0
- net USART1_TX: track 32.8 -> 0.00 mm
- net N$19: track 32.5 -> 0.00 mm, vias 5 -> 0
- net SMB0_SCL: track 29.0 -> 0.00 mm, vias 1 -> 0
- net SMB0_SDA: track 27.3 -> 0.00 mm, vias 3 -> 0
- net SPI1_MOSI: track 26.6 -> 0.00 mm
- net SPI1_CS: track 25.5 -> 0.00 mm, vias 2 -> 0
- net IMU_SCK: track 21.8 -> 0.00 mm, vias 2 -> 0
- net GND: track 20.5 -> 0.00 mm, vias 22 -> 0
- net SPI1_SCLK: track 18.9 -> 0.00 mm, vias 2 -> 0
- net SWDCLK: track 18.9 -> 0.00 mm
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- removed copper zone on layer 16, net AGND
- removed copper zone on layer 1, net GND
- removed copper zone on layer 16, net GND
Other:
- outline, holes or cut-outs redrawn
- board text removed: "*SUGOI*"
- board text removed: "Rev.A"
- board text removed: "Sylphide technology inside"
- board text removed: "by fenrir"

Commit message: Minor update
Parts:
- removed R13, R14: 10k, mami_pero:1005
- removed U$1: LTC3550, mami_pero:DFN-16
- removed U$10: NEO-6, mami_pero:NEO-6
- removed U$11: LQG15HS, mami_pero:LQG15HS
- removed U$12: HIROSE_H.FL, mami_pero:HIROSE_H.FL
- removed U$13: JST_SH_12, mami_pero:JST_SH_12
- removed U$14: OMRON_B3U_1000P, mami_pero:B3U_1000P
- removed U$16: 2200p, mami_pero:1005
- removed U$17, U$18, U$19, U$23, U$24, U$25, U$27, U$28: 0.1u, mami_pero:1005
- removed U$2: 2.2u, mami_pero:LQH32CN
- removed U$20: pull-down, mami_pero:1005
- removed U$21: 10, mami_pero:1005
- removed U$22: 0, mami_pero:1005
- removed U$26: 1u, mami_pero:1005
- removed U$29: 3216(CAP), mami_pero:3216
- removed U$3: JST_ZR_2, mami_pero:JST_ZR_2
- removed U$30: 4.7u, mami_pero:2012
- removed U$31: 330k, mami_pero:1608
- removed U$32, U$33: 1608(LED), mami_pero:1608
- removed U$36: FA128, mami_pero:FA128
- removed U$4: MICRO_USB, mami_pero:MICRO_USB
- removed U$5: DM3A, mami_pero:DM3A
- removed U$7: MS5611-01BA03, mami_pero:MS5611
- removed U$9: STM32F405_64, mami_pero:TQFP-64
- added C14, C15, C17, C18, C19, C20, C22, C24: 0.1u, additional:1005
- added C16: 1u, additional:1005
- added C21, C23: 2.2u, additional:1005
- added CON1: (no value), additional:JST_ZH-2B(MM)
- added CON2: ZX62-B-5PA(11), additional:ZX62-AB-5PA
- added CON3: JST_SH-12SM, additional:JST_SH-SM12B
- added IC1: LTC3550EDHC, main:DFN16BP
- added IC2: MPU-6000, sensor:QFN24
- added IC4: MAG3110FCR, main:DFN10
- added J1: JUMPER1608, additional:1608
- added L1: 2.2u, additional:3225
- added L2: LQG15HS27NJ02, additional:1005
- added LED3: LED3, mami_pero:1608
- added LED4: 1608(LED), mami_pero:1608
- added R10, R11: 10K, additional:1005
- added R8: 10, additional:1005
- added R9: pull-down, additional:1005
- added U1: DM3AT-SF-PEJM5, additional:DM3
- added U2: H.FL, gps:H.FL
- added U3: NEO-6T, gps:NEO
- added U4: MS5611-01BA01, sensor:LGA8
- C1: value 0.1u -> 10u; device mami_pero:1005 -> additional:3216
- C10, C11: value 8p -> 0.1u; device mami_pero:1005 -> additional:1005
- C12, C13: value 0,1u -> 0.1u; device mami_pero:1005 -> additional:1005
- C2, C3, C5, C6: device mami_pero:1005 -> additional:1005
- C4: value 0.1u -> 4.7u; device mami_pero:1005 -> additional:2012
- C7: value 0,1u -> 2200p; device mami_pero:1005 -> additional:1005
- C8, C9: value 2.2u -> 0.1u; device mami_pero:1005 -> additional:1005
- LED1, LED2: value 1608(LED) -> (none); device mami_pero:1608 -> additional:1608D
- R1, R2: value 1k -> 1K; device mami_pero:1005 -> additional:1005
- R3, R4: value 2k -> 2K; device mami_pero:1005 -> additional:1005
- R5: value 1.24k -> 1.24K; device mami_pero:1005 -> additional:1005
- R6: value 604k -> 604K; device mami_pero:1005 -> additional:1005
- R7: value 150k -> 150K; device mami_pero:1005 -> additional:1005
- U$15: value 0.1u -> 330k
- U$6: value MPU6000 -> STM32F405_64; device mami_pero:QFN24 -> mami_pero:TQFP-64
- U$8: value MAG3110 -> OMRON_B3U_1000P; device mami_pero:MAG3110 -> mami_pero:B3U_1000P
- moved C9 85.0 mm to (24.0, 6.91), flipped to the bottom
- moved C13 84.9 mm to (19.9, 25.2), flipped to the bottom, turned to 90 degrees
- moved C11 77.2 mm to (20.0, 13.8), turned to 90 degrees
- moved C10 77.1 mm to (22.9, 5.28), flipped to the bottom
- moved C7 76.4 mm to (22.4, 8.24), flipped to the bottom, turned to 270 degrees
- moved C12 76.2 mm to (16.1, 17.4)
- moved C4 62.8 mm to (17.4, 8.84), flipped to the bottom
- moved C8 61.5 mm to (2.65, 11.6), flipped to the bottom, turned to 180 degrees
- moved C6 61.2 mm to (13.7, 16.9)
- moved U$35 59.5 mm to (1.98, 11.8), turned to 90 degrees
- moved U$6 59.2 mm to (18.3, 5.99), turned to 90 degrees
- moved U$34 58.1 mm to (1.98, 9.10), turned to 90 degrees
- moved U$15 56.9 mm to (21.9, 15.6), turned to 270 degrees
- moved U$8 55.6 mm to (23.5, 14.2), turned to 90 degrees
- moved C1 54.3 mm to (22.0, 14.0), flipped to the bottom, turned to 270 degrees
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Connections:
- removed net +3V3: C1.P$2, C12.P$2, C13.P$2, C4.P$2, C5.P$2, C6.P$2, C7.P$2, R13.P$2, R14.P$2, R6.P$2, U$10.23, U$15.P$2, U$18.P$2, U$19.P$2, U$2.P$2, U$25.P$2, U$26.P$2, U$27.P$2, U$28.P$2, U$29.P$2, U$31.P$2, U$5.4, U$6.13, U$7.P$1, U$7.P$2, U$8.P$2, U$8.P$8, U$9.P$1, U$9.P$13, U$9.P$19, U$9.P$32, U$9.P$48, U$9.P$64
- removed net +5V: C2.P$2, U$1.1, U$4.1
- removed net -INT: U$10.3
- removed net AUX_MAG_SCL: R14.P$1, U$6.7, U$7.P$8, U$8.P$7
- removed net AUX_MAG_SDA: R13.P$1, U$6.6, U$7.P$7, U$8.P$6
- removed net GPS_USB_VBAS: U$10.7, U$20.P$2
- removed net IMU_INTR: U$6.12
- removed net IMU_SCLK: U$6.23, U$9.P$21
- removed net N$23: C10.P$2, U$36.1, U$9.P$5
- removed net N$24: C11.P$2, U$36.3, U$9.P$6
- removed net SPI3_CS: U$5.2, U$9.P$50
- removed net SPI3_MISO: U$5.7, U$9.P$52
- removed net SPI3_MOSI: U$5.3, U$9.P$53
- removed net SPI3_SCK: U$5.5, U$9.P$51
- new net +3V: C1.2, C11.P$1, C12.P$1, C15.P$2, C16.P$2, C17.P$2, C18.P$1, C19.P$1, C20.P$2, C22.P$1, C24.P$1, C5.P$2, C6.P$2, C8.P$2, C9.P$1, CON3.3, IC2.13, IC4.2, IC4.8, L1.2, R10.P$1, R11.P$1, R6.P$1, U$15.P$2, U$6.P$1, U$6.P$13, U$6.P$19, U$6.P$32, U$6.P$48, U$6.P$64, U1.4, U3.23, U4.1, U4.2
- new net -INT0: U$6.P$26, U3.3
- new net GPS_USB_VBUS: R9.P$2, U3.7
- new net IMU_-CS: IC2.8
- new net IMU_SCK: IC2.23, U$6.P$51
- new net INT_MPU: IC2.12, U$6.P$2
- new net SMB0_SCL: IC2.7, IC4.7, R11.P$2, U4.8
- new net SMB0_SDA: IC2.6, IC4.6, R10.P$2, U4.7
- new net SPI1_CS: U$6.P$20, U1.2
- new net SPI1_MISO: U$6.P$22, U1.7
- new net SPI1_MOSI: U$6.P$23, U1.3
- new net SPI1_SCLK: U$6.P$21, U1.5
- new net USB_VBUS: C2.P$2, CON2.1, IC1.1
- net AGND: now also J1.P$1, U2.GND@1, U2.GND@2, U2.GND@3, U3.10, U3.12, U3.13; no longer U$10.10, U$10.12, U$10.24, U$12.GND@1, U$12.GND@2, U$12.GND@3, U$22.P$1
- net GND: now also C1.1, C10.P$2, C11.P$2, C12.P$2, C14.P$1, C15.P$1, C16.P$1, C17.P$1, C18.P$2, C19.P$2, C20.P$1, C21.P$1, C22.P$2, C23.P$1, C24.P$2, C3.P$2, C4.1, C7.P$2, C9.P$2, CON1.2, CON2.5, CON2.GUIDE@L1, CON2.GUIDE@L3, CON2.GUIDE@R1, CON2.GUIDE@R3, CON3.2, CON3.4, CON3.GUIDE@L, CON3.GUIDE@R, IC1.17, IC1.8, IC1.9, IC2.1, IC2.11, IC2.18, IC4.10, IC4.5, J1.P$2, R3.P$2, R4.P$2, R5.P$2, R7.P$2, R9.P$1, U$6.P$12, U$6.P$18, U$6.P$63, U$8.P$1, U1.6, U1.GND@1, U1.GND@2, U1.GND@3, U1.GND@4, U3.24, U4.3, U4.4; no longer C1.P$1, C10.P$1, C11.P$1, C12.P$1, C3.P$1, C4.P$1, C7.P$1, C9.P$1, R3.P$1, R4.P$1, R5.P$1, R7.P$1, U$1.8, U$1.9, U$1.P$17, U$10.13, U$14.P$1, U$15.P$1, U$16.P$1, U$18.P$1, U$19.P$1, U$20.P$1, U$22.P$2, U$23.P$1, U$24.P$1, U$25.P$1, U$26.P$1, U$27.P$1, U$28.P$1, U$29.P$1, U$3.P$1, U$30.1, U$4.5, U$5.6, U$5.GND@1, U$5.GND@2, U$5.GND@3, U$5.GND@4, U$6.1, U$6.11, U$6.18, U$7.P$3, U$7.P$4, U$8.P$10, U$8.P$5, U$9.P$12, U$9.P$18, U$9.P$63
- net GPIO1: now also U$6.P$24; no longer U$9.P$24
- net GPIO2: now also U$6.P$25; no longer U$9.P$25
- net GPS_BKUP: now also U3.22; no longer U$10.22
- net GPS_RX: now also U$6.P$38, U3.20; no longer U$10.20, U$9.P$38
- net GPS_TX: now also U$6.P$37, U3.21; no longer U$10.21, U$9.P$37
- net GPS_USB_D+: now also U3.6; no longer U$10.6
- net GPS_USB_D-: now also U3.5; no longer U$10.5
- net I2C1_SCL: now also CON3.6, U$6.P$61; no longer U$9.P$61
- net I2C1_SDA: now also CON3.5, U$6.P$62; no longer U$9.P$62
- net I2C2_SCL: now also U$6.P$29; no longer U$9.P$29
- net I2C2_SDA: now also U$6.P$30; no longer U$9.P$30
- net IMU_CS: now also U$6.P$50; no longer U$6.8, U$9.P$20
- net IMU_MISO: now also IC2.9, U$6.P$52; no longer U$6.9, U$9.P$22
- net IMU_MOSI: now also IC2.24, U$6.P$53; no longer U$6.24, U$9.P$23
- net N$1: now also C10.P$1, IC2.10; no longer U$1.10, U$2.P$1
- net N$10: now also LED4.P$2, U$35.P$2; no longer LED2.P$2, R2.P$2
- net N$11: now also LED2.K, R2.P$1; no longer U$33.P$1, U$9.P$35
- net N$12: now also IC1.2, R3.P$1; no longer U$32.P$2, U$34.P$2
- net N$13: now also IC1.3, R4.P$1; no longer U$16.P$2, U$6.20
- net N$14: now also IC1.14, R5.P$1; no longer U$17.P$2, U$6.10
- net N$15: now also C5.P$1, IC1.6, R6.P$2, R7.P$1; no longer U$10.11, U$11.P$2, U$12.SIG
- net N$16: now also IC1.5, R1.P$2; no longer U$24.P$2, U$8.P$4
- net N$17: now also IC1.10, L1.1; no longer U$23.P$2, U$8.P$1
- net N$18: now also IC1.4, R2.P$2; no longer U$10.8, U$10.9, U$21.P$2
- net N$19: now also C4.2, CON1.1, IC1.11, IC1.15, IC1.7, LED1.A, LED2.A; no longer U$11.P$1, U$21.P$1
- net N$2: now also C23.P$2, U$6.P$31; no longer R3.P$2, U$1.2
- net N$20: now also LED3.P$1, U$6.P$36; no longer U$32.P$1, U$9.P$36
- net N$21: now also U$15.P$1, U$6.P$7, U$8.P$2; no longer U$14.P$2, U$31.P$1, U$9.P$7
- net N$22: now also C13.P$2, IC4.1; no longer U$33.P$2, U$35.P$2
- net N$29: now also C14.P$2, IC4.4; no longer C8.P$2, U$9.P$31
- net N$3: now also C7.P$1, IC2.20; no longer R4.P$2, U$1.3
- net N$31: now also C21.P$2, U$6.P$47; no longer C9.P$2, U$9.P$47
- net N$4: now also LED4.P$1, U$6.P$35; no longer R5.P$2, U$1.14
- net N$5: now also LED3.P$2, U$34.P$2; no longer LED1.P$1, LED2.P$1, U$1.11, U$1.15, U$1.7, U$3.P$2, U$30.2
- net N$6: now also L2.P$1, R8.P$1; no longer C5.P$1, R7.P$2, U$1.6
- net N$7: now also L2.P$2, U2.SIG, U3.11; no longer R1.P$1, U$1.5
- net N$8: now also R8.P$2, U3.8, U3.9; no longer LED1.P$2, R1.P$2
- net N$9: now also LED1.K, R1.P$1; no longer R2.P$1, U$1.4
- net SWDCLK: now also CON3.11, U$6.P$49; no longer U$9.P$49
- net SWDIO: now also CON3.12, U$6.P$46; no longer U$9.P$46
- net USART1_RX: now also CON3.8, U$6.P$59; no longer U$9.P$59
- net USART1_TX: now also CON3.7, U$6.P$58; no longer U$9.P$58
- net USB_D+: now also CON2.3, U$6.P$45; no longer U$4.3, U$9.P$45
- net USB_D-: now also CON2.2, U$6.P$44; no longer U$4.2, U$9.P$44
- net USB_ID: now also CON2.4; no longer U$4.4
- net VCC: now also C3.P$1, CON3.1, IC1.16; no longer C3.P$2, U$1.16
Routing:
- net +3V: track 0.00 -> 166.2 mm, vias 0 -> 13
- net VCC: track 0.00 -> 57.5 mm, vias 0 -> 3
- net I2C1_SDA: track 0.00 -> 41.0 mm
- net I2C1_SCL: track 0.00 -> 39.8 mm
- net USART1_RX: track 0.00 -> 34.2 mm, vias 0 -> 2
- net USART1_TX: track 0.00 -> 32.9 mm
- net N$19: track 0.00 -> 32.8 mm, vias 0 -> 5
- net SMB0_SCL: track 0.00 -> 28.7 mm, vias 0 -> 1
- net SMB0_SDA: track 0.00 -> 28.1 mm, vias 0 -> 3
- net SPI1_MOSI: track 0.00 -> 26.7 mm
- net SPI1_CS: track 0.00 -> 25.5 mm, vias 0 -> 2
- net IMU_SCK: track 0.00 -> 22.9 mm, vias 0 -> 2
- net GND: track 0.00 -> 22.7 mm, vias 0 -> 31
- net -INT0: track 0.00 -> 20.9 mm, vias 0 -> 1
- net SWDCLK: track 0.00 -> 20.0 mm
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- added copper zone on layer 16, net AGND
- added copper zone on layer 1, net GND
- added copper zone on layer 16, net GND
Other:
- outline, holes or cut-outs redrawn
- board text added: "*SUGOI*"
- board text added: "Rev.A"
- board text added: "Sylphide technology inside"
- board text added: "by fenrir"

Commit message: Bug fixed
Parts:
- removed U$15: 330k, mami_pero:1005
- added R12: 330k, mami_pero:1005
- moved C19 1.84 mm to (7.10, 3.50), turned to 270 degrees
- moved U4 1.00 mm to (23.0, 25.6)
- renumbered U$34 to R13, U$35 to R14
Connections:
- net +3V: now also R12.P$2; no longer U$15.P$2
- net N$21: now also R12.P$1; no longer U$15.P$1
Routing:
- net GND: track 22.7 -> 20.2 mm
- net +3V: track 166.2 -> 168.5 mm
- net SMB0_SCL: track 28.7 -> 29.6 mm
- net SMB0_SDA: track 28.1 -> 28.8 mm
- net USART1_RX: track 34.2 -> 34.8 mm
- net USART1_TX: track 32.9 -> 33.5 mm
- net I2C1_SCL: track 39.8 -> 40.3 mm
Other:
- board text removed: "*SUGOI*"
- board text removed: "Rev.A"
- board text removed: "Sylphide technology inside"
- board text removed: "by fenrir"
