File: NinjaScanPseudo.sch (EAGLE design)
At the start: 57 parts, among them CON2 ZX62-B-5PA(11), CON3 JST_SH-12SM, IC1 LTC3550EDHC, IC2 MPU-6000, IC4 MAG3110FCR, J1 JUMPER1608, U1 DM3AT-SF-PEJM5, U2 H.FL, U3 NEO-6T, U4 MS5611-01BA01

Commit message: some wiring issues were fixed.
Parts:
- removed C14, C15, C17, C18, C19, C20, C22, C24: 0.1u, additional:C1005
- removed C16: 1u, additional:C1005
- removed C21, C23: 2.2u, additional:C1005
- removed CON1: (no value), additional:JST_ZH-2B(MM)
- removed CON2: ZX62-B-5PA(11), additional:ZX62-AB-5PA
- removed CON3: JST_SH-12SM, additional:JST_SH-12SM
- removed IC1: LTC3550EDHC, main:LTC3550EDHC
- removed IC2: MPU-6000, sensor:MPU-6000
- removed IC4: MAG3110FCR, main:MAG3110FCR
- removed J1: JUMPER1608, additional:JUMPER1608
- removed L1: 2.2u, additional:L3225
- removed L2: LQG15HS27NJ02, additional:L1005
- removed LED3: LED3, mami_pero:1608(LED)
- removed LED4: 1608(LED), mami_pero:1608(LED)
- removed R10, R11: 10K, additional:R1005
- removed R8: 10, additional:R1005
- removed R9: pull-down, additional:R1005
- removed U1: DM3AT-SF-PEJM5, additional:DM3A-SF-PEJ2
- removed U2: H.FL, gps:H.FL
- removed U3: NEO-6T, gps:NEO-6T
- removed U4: MS5611-01BA01, sensor:MS5611-01BA01
- added R13, R14: 10k, mami_pero:1005(RES)
- added U$1: LTC3550, mami_pero:LTC3550
- added U$10: NEO-6, mami_pero:NEO-6
- added U$11: LQG15HS, mami_pero:LQG15HS
- added U$12: HIROSE_H.FL, mami_pero:HIROSE_H.FL
- added U$13: JST_SH_12, mami_pero:JST_SH_12
- added U$14: OMRON_B3U_1000P, mami_pero:OMRON_B3U_1000P
- added U$16: 2200p, mami_pero:1005(CAP)
- added U$17, U$18, U$19, U$23, U$24, U$25, U$27, U$28: 0.1u, mami_pero:1005(CAP)
- added U$2: 2.2u, mami_pero:LQH32CN
- added U$20: pull-down, mami_pero:1005(RES)
- added U$21: 10, mami_pero:1005(RES)
- added U$22: 0, mami_pero:1005(RES)
- added U$26: 1u, mami_pero:1005(CAP)
- added U$29: 3216(CAP), mami_pero:3216(CAP)
- added U$3: JST_ZR_2, mami_pero:JST_ZR_2
- added U$30: 4.7u, mami_pero:2012(CAP)
- added U$31: 330k, mami_pero:1608(RES)
- added U$32, U$33: 1608(LED), mami_pero:1608(LED)
- added U$36: FA128, mami_pero:FA128
- added U$4: MICRO_USB, mami_pero:MICRO_USB
- added U$5: DM3A, mami_pero:DM3A
- added U$7: MS5611-01BA03, mami_pero:MS5611-01BA03
- added U$9: STM32F405_64, mami_pero:STM32F405_64
- C1: value 10u -> 0.1u; device additional:C3216 -> mami_pero:1005(CAP)
- C10, C11: value 0.1u -> 8p; device additional:C1005 -> mami_pero:1005(CAP)
- C12, C13: value 0.1u -> 0,1u; device additional:C1005 -> mami_pero:1005(CAP)
- C2, C3, C5, C6: device additional:C1005 -> mami_pero:1005(CAP)
- C4: value 4.7u -> 0.1u; device additional:C2012 -> mami_pero:1005(CAP)
- C7: value 2200p -> 0,1u; device additional:C1005 -> mami_pero:1005(CAP)
- C8, C9: value 0.1u -> 2.2u; device additional:C1005 -> mami_pero:1005(CAP)
- LED1, LED2: value (none) -> 1608(LED); device additional:LED1608 -> mami_pero:1608(LED)
- R1, R2: value 1K -> 1k; device additional:R1005 -> mami_pero:1005(RES)
- R3, R4: value 2K -> 2k; device additional:R1005 -> mami_pero:1005(RES)
- R5: value 1.24K -> 1.24k; device additional:R1005 -> mami_pero:1005(RES)
- R6: value 604K -> 604k; device additional:R1005 -> mami_pero:1005(RES)
- R7: value 150K -> 150k; device additional:R1005 -> mami_pero:1005(RES)
- U$15: value 330k -> 0.1u; device mami_pero:1005(RES) -> mami_pero:1005(CAP)
- U$6: value STM32F405_64 -> MPU6000; device mami_pero:STM32F405_64 -> mami_pero:MPU6000
- U$8: value OMRON_B3U_1000P -> MAG3110; device mami_pero:OMRON_B3U_1000P -> mami_pero:MAG3110
Connections:
- removed net +3V: C1.2, C11.1, C12.1, C15.2, C16.2, C17.2, C18.1, C19.1, C20.2, C22.1, C24.1, C5.2, C6.2, C8.2, C9.1, CON3.3, IC2.VDD, IC4.VDD, IC4.VDDIO, L1.2, R10.1, R11.1, R6.1, U$15.2, U$6.VBAT, U$6.VDD@1, U$6.VDD@2, U$6.VDD@3, U$6.VDD@4, U$6.VDDA, U1.VDD, U3.VCC, U4.I2C/-SPI, U4.VDD
- removed net -INT0: U3.TIMEPULSE
- removed net GPS_USB_VBUS: R9.2, U3.VDDUSB
- removed net IMU_-CS: IC2.-CS
- removed net IMU_SCK: IC2.SCL/SCLK, U$6.PC10
- removed net SMB0_SCL: IC2.AUX_CL, IC4.SCL, R11.2, U4.SCLK
- removed net SMB0_SDA: IC2.AUX_DA, IC4.SDA, R10.2, U4.SDI/SDA
- removed net SPI1_CS: U$6.PA4, U1.-CS(DAT3)
- removed net SPI1_MISO: U$6.PA6, U1.DO(DAT0)
- removed net SPI1_MOSI: U$6.PA7, U1.DI(CMD)
- removed net SPI1_SCLK: U$6.PA5, U1.SCLK
- removed net USB_VBUS: C2.2, CON2.VBUS, IC1.USBIN
- new net +3V3: C1.P$2, C12.P$2, C13.P$2, C4.P$2, C5.P$2, C6.P$2, C7.P$2, R13.2, R14.2, R6.2, U$10.VCC@1, U$15.P$2, U$18.P$2, U$19.P$2, U$2.P$2, U$25.P$2, U$26.P$2, U$27.P$2, U$28.P$2, U$29.P$2, U$31.2, U$5.VDD, U$6.VDD, U$7.I2C/-SPI, U$7.VDD, U$8.VDD, U$8.VDDIO, U$9.VBAT, U$9.VDD@1, U$9.VDD@2, U$9.VDD@3, U$9.VDD@4, U$9.VDDA
- new net +5V: C2.P$2, U$1.USBIN, U$4.VCC
- new net -INT: U$10.TIMEPULSE
- new net AUX_MAG_SCL: R14.1, U$6.AUXCL, U$7.SCLK, U$8.SCL
- new net AUX_MAG_SDA: R13.1, U$6.AUXDA, U$7.SDI/SDA, U$8.SDA
- new net GPS_USB_VBAS: U$10.VDDUSB, U$20.2
- new net IMU_INTR: U$6.INT
- new net IMU_SCLK: U$6.SCL/SCLK, U$9.PA5
- new net N$23: C10.P$2, U$36.P$1, U$9.PH0
- new net N$24: C11.P$2, U$36.P$2, U$9.PH1
- new net SPI3_CS: U$5.CD/DAT3, U$9.PA15
- new net SPI3_MISO: U$5.DAT0, U$9.PC11
- new net SPI3_MOSI: U$5.CMD, U$9.PC12
- new net SPI3_SCK: U$5.CLK, U$9.PC10
- net AGND: now also U$10.GND@1, U$10.GND@2, U$10.GND@4, U$12.GND, U$22.1; no longer J1.P$1, U2.GND@2, U2.GND@3, U2.GND@4, U3.GND@10, U3.GND@12, U3.GND@13
- net GND: now also C1.P$1, C10.P$1, C11.P$1, C12.P$1, C13.P$1, C2.P$1, C3.P$1, C4.P$1, C6.P$1, C7.P$1, C8.P$1, C9.P$1, R3.1, R4.1, R5.1, R7.1, U$1.GND@1, U$1.GND@2, U$1.GND@3, U$10.GND@3, U$14.P$1, U$15.P$1, U$16.P$1, U$18.P$1, U$19.P$1, U$20.1, U$22.2, U$23.P$1, U$24.P$1, U$25.P$1, U$26.P$1, U$27.P$1, U$28.P$1, U$29.P$1, U$3.P$1, U$30.P$1, U$4.GND, U$5.GND@1, U$5.GND@2, U$5.GND@3, U$5.GND@4, U$5.VSS, U$6.CLKIN, U$6.FSYNC, U$6.GND, U$7.CSB@1, U$7.GND, U$8.GND@1, U$8.GND@2, U$9.VSS@1, U$9.VSS@4, U$9.VSSA; no longer C1.1, C10.2, C11.2, C12.2, C13.1, C14.1, C15.1, C16.1, C17.1, C18.2, C19.2, C2.1, C20.1, C21.1, C22.2, C23.1, C24.2, C3.2, C4.1, C6.1, C7.2, C8.1, C9.2, CON1-2.P$1, CON2.GND, CON3.2, CON3.4, CON3.GUIDE@L, CON3.GUIDE@R, IC1.GND@17, IC1.GND@8, IC1.GND@9, IC2.CLKIN, IC2.FSYNC, IC2.GND, IC4.GND@10, IC4.GND@5, J1.P$2, R3.2, R4.2, R5.2, R7.2, R9.1, U$6.VSS@1, U$6.VSS@4, U$6.VSSA, U$8.P$1, U1.VSS, U3.GND@24, U4.CSB@4, U4.GND
- net GPIO1: now also U$9.PC4; no longer U$6.PC4
- net GPIO2: now also U$9.PC5; no longer U$6.PC5
- net GPS_BKUP: now also U$10.V_BKUP; no longer U3.V_BCKP
- net GPS_RX: now also U$10.TXD1, U$9.PC7; no longer U$6.PC7, U3.TXD1
- net GPS_TX: now also U$10.RXD1, U$9.PC6; no longer U$6.PC6, U3.RXD1
- net GPS_USB_D+: now also U$10.D+; no longer U3.USB_DP
- net GPS_USB_D-: now also U$10.D-; no longer U3.USB_DM
- net I2C1_SCL: now also U$9.PB8; no longer CON3.6, U$6.PB8
- net I2C1_SDA: now also U$9.PB9; no longer CON3.5, U$6.PB9
- net I2C2_SCL: now also U$9.PB10; no longer U$6.PB10
- net I2C2_SDA: now also U$9.PB11; no longer U$6.PB11
- net IMU_CS: now also U$6.CS, U$9.PA4; no longer U$6.PA15
- net IMU_MISO: now also U$6.AD0/SDO, U$9.PA6; no longer IC2.AD0/SDO, U$6.PC11
- net IMU_MOSI: now also U$6.SDA/SDI, U$9.PA7; no longer IC2.SDA/SDI, U$6.PC12
- net N$1: now also U$1.SW, U$2.P$1; no longer C10.1, IC2.REGOUT
- net N$10: now also LED2.P$2, R2.2; no longer LED4.P$2, U$35.2
- net N$11: now also U$33.P$1, U$9.PB14; no longer LED2.K, R2.1
- net N$12: now also U$32.P$2, U$34.2; no longer IC1.IUSB, R3.1
- net N$13: now also U$16.P$2, U$6.CPOUT; no longer IC1.ITERM, R4.1
- net N$14: now also U$17.P$2, U$6.REGOUT; no longer IC1.IDC, R5.1
- net N$15: now also U$10.RF_IN, U$11.P$2, U$12.SIG; no longer C5.1, IC1.VFB, R6.2, R7.1
- net N$16: now also U$24.P$2, U$8.CAP-R; no longer IC1.-CHRG, R1.2
- net N$17: now also U$23.P$2, U$8.CAP-A; no longer IC1.SW, L1.1
- net N$18: now also U$10.RESERVED@2, U$10.VCC_RF, U$21.2; no longer IC1.-PWR, R2.2
- net N$19: now also U$11.P$1, U$21.1; no longer C4.2, CON1-1.P$1, IC1.BAT, IC1.RUN, IC1.VCC, LED1.A, LED2.A
- net N$2: now also R3.2, U$1.IUSB; no longer C23.2, U$6.VCAP_1
- net N$20: now also U$32.P$1, U$9.PB15; no longer LED3.P$1, U$6.PB15
- net N$21: now also U$14.P$2, U$31.1, U$9.NRST; no longer U$15.1, U$6.NRST, U$8.P$2
- net N$22: now also U$33.P$2, U$35.2; no longer C13.2, IC4.CAP-A
- net N$29: now also C8.P$2, U$9.VCAP_1; no longer C14.2, IC4.CAP-R
- net N$3: now also R4.2, U$1.ITERM; no longer C7.1, IC2.CPOUT
- net N$31: now also C9.P$2, U$9.VCAP_2; no longer C21.2, U$6.VCAP_2
- net N$4: now also R5.2, U$1.IDC; no longer LED4.P$1, U$6.PB14
- net N$5: now also LED1.P$1, LED2.P$1, U$1.BAT, U$1.RUN, U$1.VCC, U$3.P$2, U$30.P$2; no longer LED3.P$2, U$34.2
- net N$6: now also C5.P$1, R7.2, U$1.VFB; no longer L2.1, R8.1
- net N$7: now also R1.1, U$1.-CHRG; no longer L2.2, U2.C, U3.RF_IN
- net N$8: now also LED1.P$2, R1.2; no longer R8.2, U3.RESERVED@8, U3.VCC_RF
- net N$9: now also R2.1, U$1.-PWR; no longer LED1.K, R1.1
- net SWDCLK: now also U$9.PA14; no longer CON3.11, U$6.PA14
- net SWDIO: now also U$9.PA13; no longer CON3.12, U$6.PA13
- net USART1_RX: now also U$9.PB7; no longer CON3.8, U$6.PB7
- net USART1_TX: now also U$9.PB6; no longer CON3.7, U$6.PB6
- net USB_D+: now also U$4.D+, U$9.PA12; no longer CON2.D+, U$6.PA12
- net USB_D-: now also U$4.D-, U$9.PA11; no longer CON2.D-, U$6.PA11
- net USB_ID: now also U$4.NC; no longer CON2.ID
- net VCC: now also C3.P$2, U$1.DCIN; no longer C3.1, CON3.1, IC1.DCIN
Other:
- note added: "IC1 LTC3550"
- note added: "IC3 MPU6000"
- note added: "IC4 MS5611"
- note added: "IC5 MAG3110"
- note added: "IC6 ublox NEO Series"
- note removed: "455-1812-1-ND"
- note removed: "490-2628-1-ND"
- note removed: "490-4056-1-ND"
- note removed: "For Battery"
- note removed: "H11634CT-ND"
- note removed: "LQH32CN"
- moved on the sheet: C1, C10, C11, C12, C13, C2, C3, C4, C5, C6, C7, C8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

Commit message: Minor update
Parts:
- removed R13, R14: 10k, mami_pero:1005(RES)
- removed U$1: LTC3550, mami_pero:LTC3550
- removed U$10: NEO-6, mami_pero:NEO-6
- removed U$11: LQG15HS, mami_pero:LQG15HS
- removed U$12: HIROSE_H.FL, mami_pero:HIROSE_H.FL
- removed U$13: JST_SH_12, mami_pero:JST_SH_12
- removed U$14: OMRON_B3U_1000P, mami_pero:OMRON_B3U_1000P
- removed U$16: 2200p, mami_pero:1005(CAP)
- removed U$17, U$18, U$19, U$23, U$24, U$25, U$27, U$28: 0.1u, mami_pero:1005(CAP)
- removed U$2: 2.2u, mami_pero:LQH32CN
- removed U$20: pull-down, mami_pero:1005(RES)
- removed U$21: 10, mami_pero:1005(RES)
- removed U$22: 0, mami_pero:1005(RES)
- removed U$26: 1u, mami_pero:1005(CAP)
- removed U$29: 3216(CAP), mami_pero:3216(CAP)
- removed U$3: JST_ZR_2, mami_pero:JST_ZR_2
- removed U$30: 4.7u, mami_pero:2012(CAP)
- removed U$31: 330k, mami_pero:1608(RES)
- removed U$32, U$33: 1608(LED), mami_pero:1608(LED)
- removed U$36: FA128, mami_pero:FA128
- removed U$4: MICRO_USB, mami_pero:MICRO_USB
- removed U$5: DM3A, mami_pero:DM3A
- removed U$7: MS5611-01BA03, mami_pero:MS5611-01BA03
- removed U$9: STM32F405_64, mami_pero:STM32F405_64
- added C14, C15, C17, C18, C19, C20, C22, C24: 0.1u, additional:C1005
- added C16: 1u, additional:C1005
- added C21, C23: 2.2u, additional:C1005
- added CON1: (no value), additional:JST_ZH-2B(MM)
- added CON2: ZX62-B-5PA(11), additional:ZX62-AB-5PA
- added CON3: JST_SH-12SM, additional:JST_SH-12SM
- added IC1: LTC3550EDHC, main:LTC3550EDHC
- added IC2: MPU-6000, sensor:MPU-6000
- added IC4: MAG3110FCR, main:MAG3110FCR
- added J1: JUMPER1608, additional:JUMPER1608
- added L1: 2.2u, additional:L3225
- added L2: LQG15HS27NJ02, additional:L1005
- added LED3: LED3, mami_pero:1608(LED)
- added LED4: 1608(LED), mami_pero:1608(LED)
- added R10, R11: 10K, additional:R1005
- added R8: 10, additional:R1005
- added R9: pull-down, additional:R1005
- added U1: DM3AT-SF-PEJM5, additional:DM3A-SF-PEJ2
- added U2: H.FL, gps:H.FL
- added U3: NEO-6T, gps:NEO-6T
- added U4: MS5611-01BA01, sensor:MS5611-01BA01
- C1: value 0.1u -> 10u; device mami_pero:1005(CAP) -> additional:C3216
- C10, C11: value 8p -> 0.1u; device mami_pero:1005(CAP) -> additional:C1005
- C12, C13: value 0,1u -> 0.1u; device mami_pero:1005(CAP) -> additional:C1005
- C2, C3, C5, C6: device mami_pero:1005(CAP) -> additional:C1005
- C4: value 0.1u -> 4.7u; device mami_pero:1005(CAP) -> additional:C2012
- C7: value 0,1u -> 2200p; device mami_pero:1005(CAP) -> additional:C1005
- C8, C9: value 2.2u -> 0.1u; device mami_pero:1005(CAP) -> additional:C1005
- LED1, LED2: value 1608(LED) -> (none); device mami_pero:1608(LED) -> additional:LED1608
- R1, R2: value 1k -> 1K; device mami_pero:1005(RES) -> additional:R1005
- R3, R4: value 2k -> 2K; device mami_pero:1005(RES) -> additional:R1005
- R5: value 1.24k -> 1.24K; device mami_pero:1005(RES) -> additional:R1005
- R6: value 604k -> 604K; device mami_pero:1005(RES) -> additional:R1005
- R7: value 150k -> 150K; device mami_pero:1005(RES) -> additional:R1005
- U$15: value 0.1u -> 330k; device mami_pero:1005(CAP) -> mami_pero:1005(RES)
- U$6: value MPU6000 -> STM32F405_64; device mami_pero:MPU6000 -> mami_pero:STM32F405_64
- U$8: value MAG3110 -> OMRON_B3U_1000P; device mami_pero:MAG3110 -> mami_pero:OMRON_B3U_1000P
Connections:
- removed net +3V3: C1.P$2, C12.P$2, C13.P$2, C4.P$2, C5.P$2, C6.P$2, C7.P$2, R13.2, R14.2, R6.2, U$10.VCC@1, U$15.P$2, U$18.P$2, U$19.P$2, U$2.P$2, U$25.P$2, U$26.P$2, U$27.P$2, U$28.P$2, U$29.P$2, U$31.2, U$5.VDD, U$6.VDD, U$7.I2C/-SPI, U$7.VDD, U$8.VDD, U$8.VDDIO, U$9.VBAT, U$9.VDD@1, U$9.VDD@2, U$9.VDD@3, U$9.VDD@4, U$9.VDDA
- removed net +5V: C2.P$2, U$1.USBIN, U$4.VCC
- removed net -INT: U$10.TIMEPULSE
- removed net AUX_MAG_SCL: R14.1, U$6.AUXCL, U$7.SCLK, U$8.SCL
- removed net AUX_MAG_SDA: R13.1, U$6.AUXDA, U$7.SDI/SDA, U$8.SDA
- removed net GPS_USB_VBAS: U$10.VDDUSB, U$20.2
- removed net IMU_INTR: U$6.INT
- removed net IMU_SCLK: U$6.SCL/SCLK, U$9.PA5
- removed net N$23: C10.P$2, U$36.P$1, U$9.PH0
- removed net N$24: C11.P$2, U$36.P$2, U$9.PH1
- removed net SPI3_CS: U$5.CD/DAT3, U$9.PA15
- removed net SPI3_MISO: U$5.DAT0, U$9.PC11
- removed net SPI3_MOSI: U$5.CMD, U$9.PC12
- removed net SPI3_SCK: U$5.CLK, U$9.PC10
- new net +3V: C1.2, C11.1, C12.1, C15.2, C16.2, C17.2, C18.1, C19.1, C20.2, C22.1, C24.1, C5.2, C6.2, C8.2, C9.1, CON3.3, IC2.VDD, IC4.VDD, IC4.VDDIO, L1.2, R10.1, R11.1, R6.1, U$15.2, U$6.VBAT, U$6.VDD@1, U$6.VDD@2, U$6.VDD@3, U$6.VDD@4, U$6.VDDA, U1.VDD, U3.VCC, U4.I2C/-SPI, U4.VDD
- new net -INT0: U$6.PB0, U3.TIMEPULSE
- new net GPS_USB_VBUS: R9.2, U3.VDDUSB
- new net IMU_-CS: IC2.-CS
- new net IMU_SCK: IC2.SCL/SCLK, U$6.PC10
- new net INT_MPU: IC2.INT, U$6.PC13
- new net SMB0_SCL: IC2.AUX_CL, IC4.SCL, R11.2, U4.SCLK
- new net SMB0_SDA: IC2.AUX_DA, IC4.SDA, R10.2, U4.SDI/SDA
- new net SPI1_CS: U$6.PA4, U1.-CS(DAT3)
- new net SPI1_MISO: U$6.PA6, U1.DO(DAT0)
- new net SPI1_MOSI: U$6.PA7, U1.DI(CMD)
- new net SPI1_SCLK: U$6.PA5, U1.SCLK
- new net USB_VBUS: C2.2, CON2.VBUS, IC1.USBIN
- net AGND: now also J1.P$1, U2.GND@2, U2.GND@3, U2.GND@4, U3.GND@10, U3.GND@12, U3.GND@13; no longer U$10.GND@1, U$10.GND@2, U$10.GND@4, U$12.GND, U$22.1
- net GND: now also C1.1, C10.2, C11.2, C12.2, C13.1, C14.1, C15.1, C16.1, C17.1, C18.2, C19.2, C2.1, C20.1, C21.1, C22.2, C23.1, C24.2, C3.2, C4.1, C6.1, C7.2, C8.1, C9.2, CON1-2.P$1, CON2.GND, CON3.2, CON3.4, CON3.GUIDE@L, CON3.GUIDE@R, IC1.GND@17, IC1.GND@8, IC1.GND@9, IC2.CLKIN, IC2.FSYNC, IC2.GND, IC4.GND@10, IC4.GND@5, J1.P$2, R3.2, R4.2, R5.2, R7.2, R9.1, U$6.VSS@1, U$6.VSS@4, U$6.VSSA, U$8.P$1, U1.VSS, U3.GND@24, U4.CSB@4, U4.GND; no longer C1.P$1, C10.P$1, C11.P$1, C12.P$1, C13.P$1, C2.P$1, C3.P$1, C4.P$1, C6.P$1, C7.P$1, C8.P$1, C9.P$1, R3.1, R4.1, R5.1, R7.1, U$1.GND@1, U$1.GND@2, U$1.GND@3, U$10.GND@3, U$14.P$1, U$15.P$1, U$16.P$1, U$18.P$1, U$19.P$1, U$20.1, U$22.2, U$23.P$1, U$24.P$1, U$25.P$1, U$26.P$1, U$27.P$1, U$28.P$1, U$29.P$1, U$3.P$1, U$30.P$1, U$4.GND, U$5.GND@1, U$5.GND@2, U$5.GND@3, U$5.GND@4, U$5.VSS, U$6.CLKIN, U$6.FSYNC, U$6.GND, U$7.CSB@1, U$7.GND, U$8.GND@1, U$8.GND@2, U$9.VSS@1, U$9.VSS@4, U$9.VSSA
- net GPIO1: now also U$6.PC4; no longer U$9.PC4
- net GPIO2: now also U$6.PC5; no longer U$9.PC5
- net GPS_BKUP: now also U3.V_BCKP; no longer U$10.V_BKUP
- net GPS_RX: now also U$6.PC7, U3.TXD1; no longer U$10.TXD1, U$9.PC7
- net GPS_TX: now also U$6.PC6, U3.RXD1; no longer U$10.RXD1, U$9.PC6
- net GPS_USB_D+: now also U3.USB_DP; no longer U$10.D+
- net GPS_USB_D-: now also U3.USB_DM; no longer U$10.D-
- net I2C1_SCL: now also CON3.6, U$6.PB8; no longer U$9.PB8
- net I2C1_SDA: now also CON3.5, U$6.PB9; no longer U$9.PB9
- net I2C2_SCL: now also U$6.PB10; no longer U$9.PB10
- net I2C2_SDA: now also U$6.PB11; no longer U$9.PB11
- net IMU_CS: now also U$6.PA15; no longer U$6.CS, U$9.PA4
- net IMU_MISO: now also IC2.AD0/SDO, U$6.PC11; no longer U$6.AD0/SDO, U$9.PA6
- net IMU_MOSI: now also IC2.SDA/SDI, U$6.PC12; no longer U$6.SDA/SDI, U$9.PA7
- net N$1: now also C10.1, IC2.REGOUT; no longer U$1.SW, U$2.P$1
- net N$10: now also LED4.P$2, U$35.2; no longer LED2.P$2, R2.2
- net N$11: now also LED2.K, R2.1; no longer U$33.P$1, U$9.PB14
- net N$12: now also IC1.IUSB, R3.1; no longer U$32.P$2, U$34.2
- net N$13: now also IC1.ITERM, R4.1; no longer U$16.P$2, U$6.CPOUT
- net N$14: now also IC1.IDC, R5.1; no longer U$17.P$2, U$6.REGOUT
- net N$15: now also C5.1, IC1.VFB, R6.2, R7.1; no longer U$10.RF_IN, U$11.P$2, U$12.SIG
- net N$16: now also IC1.-CHRG, R1.2; no longer U$24.P$2, U$8.CAP-R
- net N$17: now also IC1.SW, L1.1; no longer U$23.P$2, U$8.CAP-A
- net N$18: now also IC1.-PWR, R2.2; no longer U$10.RESERVED@2, U$10.VCC_RF, U$21.2
- net N$19: now also C4.2, CON1-1.P$1, IC1.BAT, IC1.RUN, IC1.VCC, LED1.A, LED2.A; no longer U$11.P$1, U$21.1
- net N$2: now also C23.2, U$6.VCAP_1; no longer R3.2, U$1.IUSB
- net N$20: now also LED3.P$1, U$6.PB15; no longer U$32.P$1, U$9.PB15
- net N$21: now also U$15.1, U$6.NRST, U$8.P$2; no longer U$14.P$2, U$31.1, U$9.NRST
- net N$22: now also C13.2, IC4.CAP-A; no longer U$33.P$2, U$35.2
- net N$29: now also C14.2, IC4.CAP-R; no longer C8.P$2, U$9.VCAP_1
- net N$3: now also C7.1, IC2.CPOUT; no longer R4.2, U$1.ITERM
- net N$31: now also C21.2, U$6.VCAP_2; no longer C9.P$2, U$9.VCAP_2
- net N$4: now also LED4.P$1, U$6.PB14; no longer R5.2, U$1.IDC
- net N$5: now also LED3.P$2, U$34.2; no longer LED1.P$1, LED2.P$1, U$1.BAT, U$1.RUN, U$1.VCC, U$3.P$2, U$30.P$2
- net N$6: now also L2.1, R8.1; no longer C5.P$1, R7.2, U$1.VFB
- net N$7: now also L2.2, U2.C, U3.RF_IN; no longer R1.1, U$1.-CHRG
- net N$8: now also R8.2, U3.RESERVED@8, U3.VCC_RF; no longer LED1.P$2, R1.2
- net N$9: now also LED1.K, R1.1; no longer R2.1, U$1.-PWR
- net SWDCLK: now also CON3.11, U$6.PA14; no longer U$9.PA14
- net SWDIO: now also CON3.12, U$6.PA13; no longer U$9.PA13
- net USART1_RX: now also CON3.8, U$6.PB7; no longer U$9.PB7
- net USART1_TX: now also CON3.7, U$6.PB6; no longer U$9.PB6
- net USB_D+: now also CON2.D+, U$6.PA12; no longer U$4.D+, U$9.PA12
- net USB_D-: now also CON2.D-, U$6.PA11; no longer U$4.D-, U$9.PA11
- net USB_ID: now also CON2.ID; no longer U$4.NC
- net VCC: now also C3.1, CON3.1, IC1.DCIN; no longer C3.P$2, U$1.DCIN
Other:
- note added: "455-1812-1-ND"
- note added: "490-2628-1-ND"
- note added: "490-4056-1-ND"
- note added: "For Battery"
- note added: "H11634CT-ND"
- note added: "LQH32CN"
- note removed: "IC1 LTC3550"
- note removed: "IC3 MPU6000"
- note removed: "IC4 MS5611"
- note removed: "IC5 MAG3110"
- note removed: "IC6 ublox NEO Series"
- moved on the sheet: C1, C10, C11, C12, C13, C2, C3, C4, C5, C6, C7, C8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

Commit message: Bug fixed
Parts:
- renumbered U$15 to R12, U$34 to R13, U$35 to R14
Changed lines of the file:
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@@
 <part name="LED3" library="mami_pero" deviceset="1608(LED)" device="" value="LED3"/>
 <part name="LED4" library="mami_pero" deviceset="1608(LED)" device=""/>
-<part name="U$34" library="mami_pero" deviceset="1005(RES)" device=""/>
-<part name="U$35" library="mami_pero" deviceset="1005(RES)" device=""/>
+<part name="R13" library="mami_pero" deviceset="1005(RES)" device=""/>
+<part name="R14" library="mami_pero" deviceset="1005(RES)" device=""/>
 <part name="U$11" library="supply1" deviceset="+3V" device=""/>
 <part name="U$13" library="supply1" deviceset="+3V" device=""/>
-<part name="U$15" library="mami_pero" deviceset="1005(RES)" device="" value="330k"/>
+<part name="R12" library="mami_pero" deviceset="1005(RES)" device="" value="330k"/>
 <part name="C23" library="additional" deviceset="C" device="1005" value="2.2u"/>
 <part name="C21" library="additional" deviceset="C" device="1005" value="2.2u"/>
@@
 <instance part="LED3" gate="G$1" x="-40.64" y="20.32" rot="R270"/>
 <instance part="LED4" gate="G$1" x="-33.02" y="17.78" rot="R270"/>
-<instance part="U$34" gate="G$1" x="-40.64" y="-5.08" rot="R90"/>
-<instance part="U$35" gate="G$1" x="-33.02" y="-5.08" rot="R90"/>
+<instance part="R13" gate="G$1" x="-40.64" y="-5.08" rot="R90"/>
+<instance part="R14" gate="G$1" x="-33.02" y="-5.08" rot="R90"/>
 <instance part="U$11" gate="G$1" x="-111.76" y="0"/>
 <instance part="U$13" gate="G$1" x="-71.12" y="-114.3"/>
-<instance part="U$15" gate="G$1" x="-71.12" y="-132.08" rot="R90"/>
+<instance part="R12" gate="G$1" x="-71.12" y="-132.08" rot="R90"/>
 <instance part="C23" gate="G$1" x="-2.54" y="-45.72" rot="R180"/>
 <instance part="C21" gate="G$1" x="-76.2" y="-17.78" rot="R270"/>
@@
 <junction x="-40.64" y="-17.78"/>
 <junction x="-33.02" y="-17.78"/>
-<pinref part="U$34" gate="G$1" pin="1"/>
-<pinref part="U$35" gate="G$1" pin="1"/>
+<pinref part="R13" gate="G$1" pin="1"/>
+<pinref part="R14" gate="G$1" pin="1"/>
 <pinref part="C23" gate="G$1" pin="1"/>
 <pinref part="C21" gate="G$1" pin="1"/>
@@
 <wire x1="-71.12" y1="-116.84" x2="-71.12" y2="-121.92" width="0.1524" layer="91"/>
 <pinref part="U$13" gate="G$1" pin="+3V"/>
-<pinref part="U$15" gate="G$1" pin="2"/>
+<pinref part="R12" gate="G$1" pin="2"/>
 </segment>
 </net>
@@
 <wire x1="-81.026" y1="-139.7" x2="-71.12" y2="-139.7" width="0.1524" layer="91"/>
 <junction x="-81.026" y="-139.7"/>
-<pinref part="U$15" gate="G$1" pin="1"/>
+<pinref part="R12" gate="G$1" pin="1"/>
 </segment>
 </net>
@@
 <segment>
 <pinref part="LED3" gate="G$1" pin="P$2"/>
-<pinref part="U$34" gate="G$1" pin="2"/>
+<pinref part="R13" gate="G$1" pin="2"/>
 <wire x1="-40.64" y1="10.16" x2="-40.64" y2="5.08" width="0.1524" layer="91"/>
 </segment>
@@
 <segment>
 <pinref part="LED4" gate="G$1" pin="P$2"/>
-<pinref part="U$35" gate="G$1" pin="2"/>
+<pinref part="R14" gate="G$1" pin="2"/>
 <wire x1="-33.02" y1="7.62" x2="-33.02" y2="5.08" width="0.1524" layer="91"/>
 </segment>
